File: BHL S1 copied-2026-01-20_132408/_autosave-BHL S1 copied.kicad_pcb (KiCad board)
At the start: 2 copper layers, 90 parts, among them J1 Conn_01x03_Pin, J2 Conn_01x03_Pin, Q1 CSD19502Q5B, Q2 CSD19502Q5B, Q3 CSD19502Q5B, Q4 CSD19502Q5B, Q5 CSD19502Q5B, Q6 CSD19502Q5B, SW1 SW_Push, U1 ME6211C30M5, U2 SPX3819M5-L-5-0, U3 Solder Pad, U4 STM32G431CBUx, Y2 8MHz

Commit message: Net changes
Parts:
- added C29: 0.1uF, Capacitor_SMD:C_01005_0402Metric_Pad0.57x0.30mm_HandSolder, F.Cu at (31.5, 106.6)
- added C30: 0.1uF, Capacitor_SMD:C_01005_0402Metric_Pad0.57x0.30mm_HandSolder, F.Cu at (31.5, 108.2)
- added R31: 169K, Resistor_SMD:R_0402_1005Metric_Pad0.72x0.64mm_HandSolder, F.Cu at (54.4, 80.0)
- added R35: 18K, Resistor_SMD:R_0402_1005Metric_Pad0.72x0.64mm_HandSolder, F.Cu at (54.4, 86.0)
- added R36: 4.7K, Resistor_SMD:R_0402_1005Metric_Pad0.72x0.64mm_HandSolder, F.Cu at (54.4, 88.0)
- added TH1: 10K, Resistor_SMD:R_0402_1005Metric_Pad0.72x0.64mm_HandSolder, F.Cu at (54.4, 90.0)
- moved D2 101.9 mm to (65.3, 101.6)
- moved D3 101.9 mm to (65.3, 104.1)
- moved D4 101.9 mm to (65.3, 106.5)
- moved D5 101.9 mm to (65.3, 109.0)
- moved D6 101.9 mm to (65.3, 111.4)
- moved R2 99.1 mm to (31.5, 111.5)
- moved R1 99.1 mm to (31.5, 109.9)
- moved R4 99.1 mm to (31.5, 113.2)
- moved R5 99.1 mm to (31.5, 114.8)
- moved SW1 83.9 mm to (51.8, 107.5)
- moved R25 83.6 mm to (51.1, 84.0)
- moved R27 83.6 mm to (51.1, 86.0)
- moved R28 83.6 mm to (51.1, 88.0)
- moved R29 83.6 mm to (51.1, 90.0)
- moved R30 83.6 mm to (51.1, 91.9)
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Connections:
- net Net-(AS5600-SCLK) renamed SCLK
- AS5600 pad 6: Net-(AS5600-SDA) -> SDA
- Header2X2H1 pad 1: (no net) -> DCBUS
- Header2X2H1 pad 2: (no net) -> Curr_fdbk1_OPAmp-
- Header2X2H1 pad 3: (no net) -> CAN_H
- Header2X2H1 pad 4: (no net) -> CAN_L
- Header2X2H2 pad 1: (no net) -> DCBUS
- Header2X2H2 pad 2: (no net) -> Curr_fdbk1_OPAmp-
- Header2X2H2 pad 3: (no net) -> CAN_H
- Header2X2H2 pad 4: (no net) -> CAN_L
- ME3116 pad 4: Net-(ME3116-EN) -> Net-(D2-K)
- ME3116 pad 6: Net-(D2-K) -> Net-(ME3116-SW)
- R34 pad 1: Net-(AS5600-SDA) -> SDA
- R7 pad 1: Net-(ME3116-EN) -> Net-(ME3116-SW)
- U4 pad 45: B+/H2 -> SDA
Other:
- board outline added: 82 x 82 mm
