File: KiCAD Files/Protoype1_Final_revision/BHL S1 copied.kicad_sch (KiCad schematic)
At the start: 95 parts, among them IC1 NUP2105LT1G, IC2 NUP2105LT1G, IC3 IR2136STRPBF, J1 Conn_01x03_Pin, J2 Conn_01x03_Pin, Q1 CSD19502Q5B, Q2 CSD19502Q5B, Q3 CSD19502Q5B, Q4 CSD19502Q5B, Q5 CSD19502Q5B, Q7 CSD19502Q5B, U1 ME6211C30M5, U2 SPX3819M5-L-5-0, U3 Solder Pad, U4 STM32G431CBU6, Y2 8MHz

Commit message: Fixed some errors
Parts:
- AS5600: symbol Buck converter:AS5600 -> BHL_S1_CUSTOMED:AS5600
- ME3116: symbol Buck converter:ME3116 -> BHL_S1_CUSTOMED:ME3116
- TCAN1051HGVDR1: symbol Buck converter:TCAN1051HGVDR -> BHL_S1_CUSTOMED:TCAN1051HGVDR
Connections:
- net GND: now also ME3116. (EN); no longer ME3116.2 (GND)
- net at C15.2, R6.1, R8.2: now also ME3116. (EN); no longer ME3116.3 (FB)
- net at C13.1, C17.1: now also ME3116. (EN); no longer ME3116.1 (BS)
- net at C13.2, C17.2, D2.1 (K)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: now also ME3116. (EN); no longer ME3116.6 (SW)
- net at R7.1: now also ME3116. (EN); no longer ME3116.4 (EN)
- net at C16.2, D3.1 (K), R7.2: now also ME3116. (EN); no longer ME3116.5 (IN)
Other:
- moved on the sheet: TCAN1051HGVDR1
Changed lines of the file:
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@@
 	)
 	(junction
+		(at 288.29 142.24)
+		(diameter 0)
+		(color 0 0 0 0)
+	)
+	(junction
 		(at 151.13 254)
 		(diameter 0)
@@
 	)
 	(junction
-		(at 288.29 142.24)
-		(diameter 0)
-		(color 0 0 0 0)
-	)
-	(junction
 		(at 307.34 55.88)
 		(diameter 0)
@@
 	)
 	(junction
-		(at 228.6 245.11)
+		(at 284.48 144.78)
 		(diameter 0)
 		(color 0 0 0 0)
 	)
 	(junction
-		(at 280.67 121.92)
+		(at 228.6 245.11)
 		(diameter 0)
 		(color 0 0 0 0)
 	)
 	(junction
-		(at 304.8 55.88)
+		(at 280.67 121.92)
 		(diameter 0)
 		(color 0 0 0 0)
 	)
 	(junction
-		(at 66.04 173.99)
+		(at 304.8 55.88)
 		(diameter 0)
 		(color 0 0 0 0)
 	)
 	(junction
-		(at 284.48 144.78)
+		(at 66.04 173.99)
 		(diameter 0)
 		(color 0 0 0 0)
@@
 	(wire
 		(pts
-			(xy 267.97 144.78) (xy 284.48 144.78)
+			(xy 274.32 69.85) (xy 274.32 72.39)
 		)
 		(stroke
@@
 	(wire
 		(pts
-			(xy 274.32 69.85) (xy 274.32 72.39)
+			(xy 269.24 139.7) (xy 274.32 139.7)
 		)
 		(stroke
@@
 	(wire
 		(pts
+			(xy 229.87 142.24) (xy 247.65 142.24)
+		)
+		(stroke
+			(width 0)
+			(type default)
+		)
+	)
+	(wire
+		(pts
 			(xy 120.65 110.49) (xy 114.3 110.49)
 		)
@@
 	(wire
 		(pts
+			(xy 269.24 147.32) (xy 280.67 147.32)
+		)
+		(stroke
+			(width 0)
+			(type default)
+		)
+	)
+	(wire
+		(pts
 			(xy 146.05 241.3) (xy 149.86 241.3)
 		)
@@
 	(wire
 		(pts
-			(xy 267.97 142.24) (xy 288.29 142.24)
-		)
-		(stroke
-			(width 0)
-			(type default)
-		)
-	)
-	(wire
-		(pts
 			(xy 78.74 64.77) (xy 64.77 64.77)
 		)
@@
 	(wire
 		(pts
-			(xy 267.97 139.7) (xy 274.32 139.7)
-		)
-		(stroke
-			(width 0)
-			(type default)
-		)
-	)
-	(wire
-		(pts
 			(xy 332.74 101.6) (xy 314.96 101.6)
 		)
@@
 	(wire
 		(pts
-			(xy 217.17 255.27) (xy 217.17 252.73)
-		)
-		(stroke
-			(width 0)
-			(type default)
-		)
-	)
-	(wire
-		(pts
 			(xy 266.7 59.69) (xy 269.24 59.69)
 		)
@@
 	(wire
 		(pts
-			(xy 316.23 185.42) (xy 339.09 185.42)
+			(xy 238.76 147.32) (xy 247.65 147.32)
 		)
 		(stroke
@@
 	(wire
 		(pts
-			(xy 284.48 144.78) (xy 287.02 144.78)
+			(xy 316.23 185.42) (xy 339.09 185.42)
 		)
 		(stroke
@@
 	(wire
 		(pts
-			(xy 290.83 219.71) (xy 290.83 222.25)
+			(xy 284.48 144.78) (xy 287.02 144.78)
 		)
 		(stroke
@@
 	(wire
 		(pts
-			(xy 228.6 146.05) (xy 229.87 146.05)
+			(xy 290.83 219.71) (xy 290.83 222.25)
 		)
 		(stroke
@@
 	(wire
 		(pts
-			(xy 306.07 55.88) (xy 306.07 60.96)
+			(xy 228.6 146.05) (xy 229.87 146.05)
 		)
 		(stroke
@@
 	(wire
 		(pts
-			(xy 386.08 134.62) (xy 388.62 134.62)
+			(xy 306.07 55.88) (xy 306.07 60.96)
 		)
 		(stroke
@@
 	(wire
 		(pts
-			(xy 114.3 125.73) (xy 114.3 115.57)
+			(xy 386.08 134.62) (xy 388.62 134.62)
 		)
 		(stroke
@@
 	(wire
 		(pts
-			(xy 238.76 147.32) (xy 247.65 147.32)
+			(xy 114.3 125.73) (xy 114.3 115.57)
 		)
 		(stroke
@@
 	(wire
 		(pts
+			(xy 229.87 144.78) (xy 247.65 144.78)
+		)
+		(stroke
+			(width 0)
+			(type default)
+		)
+	)
+	(wire
+		(pts
 			(xy 63.5 168.91) (xy 95.25 168.91)
 		)
@@
 	(wire
 		(pts
-			(xy 280.67 147.32) (xy 267.97 147.32)
-		)
-		(stroke
-			(width 0)
-			(type default)
-		)
-	)
-	(wire
-		(pts
 			(xy 147.32 186.69) (xy 153.67 186.69)
 		)
@@
 	(wire
 		(pts
+			(xy 218.44 255.27) (xy 217.17 255.27)
+		)
+		(stroke
+			(width 0)
+			(type default)
+		)
+	)
+	(wire
+		(pts
 			(xy 372.11 31.75) (xy 372.11 36.83)
 		)
@@
 	(wire
 		(pts
-			(xy 229.87 142.24) (xy 247.65 142.24)
-		)
-		(stroke
-			(width 0)
-			(type default)
-		)
-	)
-	(wire
-		(pts
 			(xy 276.86 48.26) (xy 276.86 53.34)
 		)
@@
 	(wire
 		(pts
+			(xy 231.14 139.7) (xy 247.65 139.7)
+		)
+		(stroke
+			(width 0)
+			(type default)
+		)
+	)
+	(wire
+		(pts
 			(xy 269.24 250.19) (xy 275.59 250.19)
 		)
@@
 	(wire
 		(pts
-			(xy 217.17 252.73) (xy 182.88 252.73)
+			(xy 182.88 252.73) (xy 218.44 252.73)
 		)
 		(stroke
@@
 	(wire
 		(pts
+			(xy 269.24 142.24) (xy 288.29 142.24)
+		)
+		(stroke
+			(width 0)
+			(type default)
+		)
+	)
+	(wire
+		(pts
 			(xy 285.75 260.35) (xy 285.75 265.43)
 		)
@@
 	(wire
 		(pts
+			(xy 269.24 144.78) (xy 284.48 144.78)
+		)
+		(stroke
+			(width 0)
+			(type default)
+		)
+	)
+	(wire
+		(pts
 			(xy 269.24 265.43) (xy 281.94 265.43)
 		)
@@
 	(wire
 		(pts
-			(xy 231.14 139.7) (xy 247.65 139.7)
-		)
-		(stroke
-			(width 0)
-			(type default)
-		)
-	)
-	(wire
-		(pts
 			(xy 381 81.28) (xy 381 86.36)
 		)
@@
 	(wire
 		(pts
+			(xy 218.44 252.73) (xy 218.44 255.27)
+		)
+		(stroke
+			(width 0)
+			(type default)
+		)
+	)
+	(wire
+		(pts
 			(xy 146.05 254) (xy 151.13 254)
 		)
@@
 	(wire
 		(pts
-			(xy 229.87 144.78) (xy 247.65 144.78)
-		)
-		(stroke
-			(width 0)
-			(type default)
-		)
-	)
-	(wire
-		(pts
 			(xy 238.76 161.29) (xy 255.27 161.29)
 		)
@@
 	)
 	(symbol
-		(lib_id "Buck converter:ME3116")
+		(lib_id "BHL_S1_CUSTOMED:ME3116")
 		(at 259.08 205.74 0)
 		(unit 1)
@@
 		(dnp no)
 		(property "Reference" "ME3116"
-			(at 259.334 211.074 0)
+			(at 259.08 212.09 0)
 			(effects
 				(font
@@
 			)
 		)
-		(pin "6"
+		(pin ""
 		)
-		(pin "3"
+		(pin ""
 		)
-		(pin "2"
+		(pin ""
 		)
-		(pin "1"
+		(pin ""
 		)
-		(pin "5"
+		(pin ""
 		)
-		(pin "4"
+		(pin ""
 		)
 		(instances
@@
 	)
 	(symbol
-		(lib_id "Buck converter:TCAN1051HGVDR")
-		(at 257.81 143.51 0)
+		(lib_id "BHL_S1_CUSTOMED:TCAN1051HGVDR")
+		(at 254 143.51 0)
 		(unit 1)
 		(exclude_from_sim no)
@@
 		(on_board yes)
 		(dnp no)
-		(fields_autoplaced yes)
 		(property "Reference" "TCAN1051HGVDR1"
-			(at 257.81 133.35 0)
+			(at 258.064 134.62 0)
 			(effects
 				(font
@@
 		)
 		(property "Value" "~"
-			(at 257.81 133.35 0)
+			(at 254 133.35 0)
 			(effects
 				(font
@@
 		)
 		(property "Footprint" "Footprint for BHL S1:SOIC127P600X175-8N_CAN"
-			(at 257.81 143.51 0)
+			(at 254 143.51 0)
 			(effects
 				(font
@@
 		)
 		(property "Datasheet" ""
-			(at 257.81 143.51 0)
+			(at 254 143.51 0)
 			(effects
 				(font
@@
 		)
 		(property "Description" ""
-			(at 257.81 143.51 0)
+			(at 254 143.51 0)
 			(effects
 				(font
@@
 	)
 	(symbol
-		(lib_id "Buck converter:AS5600")
+		(lib_id "BHL_S1_CUSTOMED:AS5600")
 		(at 207.01 259.08 0)
 		(unit 1)
@@
 		(fields_autoplaced yes)
 		(property "Reference" "AS5600"
-			(at 207.01 266.192 0)
+			(at 207.01 251.46 0)
 			(effects
 				(font

Commit message: Changes to Schematic
Connections:
- net DCBUS: no longer IC3.26 (VS1)
- net SH_A: now reaches C19.2, Q1.5 (D_1), Q1.6 (D_2), Q1.7 (D_3), Q1.8 (D_4), Q1.9 (Thermo_Pad), Q7.1 (S_1), Q7.2 (S_2), Q7.3 (S_3), U3.1 (A)
- net SH_A: now also IC3.26 (VS1)
Changed lines of the file:
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@@
 	)
 	(junction
+		(at 287.02 48.26)
+		(diameter 0)
+		(color 0 0 0 0)
+	)
+	(junction
 		(at 332.74 71.12)
 		(diameter 0)
@@
 	)
 	(junction
-		(at 259.08 35.56)
-		(diameter 0)
-		(color 0 0 0 0)
-	)
-	(junction
 		(at 287.02 161.29)
 		(diameter 0)
@@
 	(wire
 		(pts
-			(xy 259.08 35.56) (xy 304.8 35.56)
+			(xy 252.73 35.56) (xy 304.8 35.56)
 		)
 		(stroke
@@
 	(wire
 		(pts
+			(xy 287.02 48.26) (xy 386.08 48.26)
+		)
+		(stroke
+			(width 0)
+			(type default)
+		)
+	)
+	(wire
+		(pts
 			(xy 275.59 48.26) (xy 276.86 48.26)
 		)
@@
 	(wire
 		(pts
+			(xy 287.02 48.26) (xy 287.02 50.8)
+		)
+		(stroke
+			(width 0)
+			(type default)
+		)
+	)
+	(wire
+		(pts
 			(xy 386.08 152.4) (xy 388.62 152.4)
 		)
@@
 	(wire
 		(pts
-			(xy 278.13 48.26) (xy 386.08 48.26)
+			(xy 278.13 48.26) (xy 287.02 48.26)
 		)
 		(stroke
@@
 	(wire
 		(pts
-			(xy 252.73 35.56) (xy 259.08 35.56)
-		)
-		(stroke
-			(width 0)
-			(type default)
-		)
-	)
-	(wire
-		(pts
 			(xy 238.76 162.56) (xy 238.76 161.29)
 		)
@@
 	(wire
 		(pts
-			(xy 259.08 39.37) (xy 259.08 35.56)
-		)
-		(stroke
-			(width 0)
-			(type default)
-		)
-	)
-	(wire
-		(pts
 			(xy 330.2 50.8) (xy 331.47 50.8)
 		)
@@
 		)
 	)
-	(global_label "SH_A"
-		(shape input)
-		(at 259.08 39.37 270)
-		(fields_autoplaced yes)
-		(effects
-			(font
-				(size 1.27 1.27)
-			)
-			(justify right)
-		)
-		(property "Intersheetrefs" "${INTERSHEET_REFS}"
-			(at 259.08 46.9514 90)
-			(effects
-				(font
-					(size 1.27 1.27)
-				)
-				(justify right)
-				(hide yes)
-			)
-		)
-	)
 	(global_label "HIN3"
 		(shape input)
@@
 				(hide yes)
 			)
+		)
+	)
+	(global_label "SH_A"
+		(shape input)
+		(at 287.02 50.8 270)
+		(fields_autoplaced yes)
+		(effects
+			(font
+				(size 1.27 1.27)
+			)
+			(justify right)
+		)
+		(property "Intersheetrefs" "${INTERSHEET_REFS}"
+			(at 287.02 58.3814 90)
+			(effects
+				(font
+					(size 1.27 1.27)
+				)
+				(justify right)
+				(hide yes)
+			)
